Commit message: same noise params for optix and embree example. removed 2d scanner from basic example

File: urdf/robot_sensor_embree.urdf.xacro (robot description, xacro)
@@ -26,9 +26,9 @@
   </collision>
   <inertial>
-      <mass value="1.0" />
+      <mass value="10.0" />
       <origin xyz="0 0 0" />
-      <inertia ixx="${0.0833333 * 1.0 * (0.3*0.3 + 0.2*0.2)}" ixy="0.0" ixz="0.0"
-        iyy="${0.0833333 * 1.0 * (0.4*0.4 + 0.2*0.2)}" iyz="0.0"
-        izz="${0.0833333 * 1.0 * (0.4*0.4 + 0.3*0.3)}" />
+      <inertia ixx="${0.0833333 * 10.0 * (0.3*0.3 + 0.2*0.2)}" ixy="0.0" ixz="0.0"
+        iyy="${0.0833333 * 10.0 * (0.4*0.4 + 0.2*0.2)}" iyz="0.0"
+        izz="${0.0833333 * 10.0 * (0.4*0.4 + 0.3*0.3)}" />
     </inertial>
 </link>
@@ -38,52 +38,4 @@
   <origin xyz="0 0 0.1" />
 </joint>
-<!-- 2D LASER -->
-<link name="laser2d">
-</link>
-<joint name="laser2d_to_base_joint" type="fixed">
-  <parent link="base_link" />
-  <child link="laser2d" />
-  <origin xyz="0 0 0.2" />
-</joint>
-<!-- <gazebo reference="laser2d">
-    <sensor type="rmagine_embree_spherical" name="laser2d">
-      <pose>0 0 0 0 0 0</pose>
-      <always_on>true</always_on>
-      <update_rate>60</update_rate>
-      <visualize>false</visualize>
-      <pre_alloc_mem>true</pre_alloc_mem>
-      <ray>
-        <scan>
-          <horizontal>
-            <min_angle>${-M_PI}</min_angle>
-            <increment>${1.0 * M_PI / 180.0}</increment>
-            <samples>360</samples>
-          </horizontal>
-        </scan>
-        <range>
-          <min>0.0</min>
-          <max>10.0</max>
-        </range>
-        <noise>
-          <type>gaussian</type>
-          <mean>0.0</mean>
-          <stddev>0.05</stddev>
-        </noise>
-      </ray>
-      <plugin name="rmagine_ros_laser2d" filename="librmagine_embree_ros_gzplugin.so">
-          <frame>laser2d</frame>
-          <outputs>
-            <output name="scan">
-              <msg>sensor_msgs/LaserScan</msg>
-              <topic>laser2d/scan</topic>
-            </output>
-            <output name="pcl">
-              <msg>sensor_msgs/PointCloud</msg>
-              <topic>laser2d/pcl</topic>
-            </output>
-          </outputs>
-      </plugin>
-    </sensor>
-</gazebo> -->
 <!-- 3D LASER -->
 <link name="laser3d">
@@ -115,23 +67,18 @@
         </scan>
         <range>
-          <min>0.0</min>
-          <max>80.0</max>
+          <min>0.2</min>
+          <max>100.0</max>
         </range>
+        <noise>
+          <type>uniform_dust</type>
+          <hit_prob>0.0000001</hit_prob>
+          <return_prob>0.5</return_prob>
+        </noise>
         <noise>
           <type>rel_gaussian</type>
           <mean>0.0</mean>
-          <stddev>0.01</stddev>
-          <range_exp>1.5</range_exp>
+          <stddev>0.002</stddev>
+          <range_exp>1.0</range_exp>
         </noise>
-        <!-- <noise>
-          <type>gaussian</type>
-          <mean>0.0</mean>
-          <stddev>0.01</stddev>
-        </noise>
-        <noise>
-          <type>uniform_dust</type>
-          <hit_prob>0.000001</hit_prob>
-          <return_prob>0.85</return_prob>
-        </noise> -->
       </ray>
       <plugin name="rmagine_ros_laser3d" filename="librmagine_embree_ros_gzplugin.so">

File: urdf/robot_sensor_optix.urdf.xacro (robot description, xacro)
@@ -26,9 +26,9 @@
   </collision>
   <inertial>
-      <mass value="1.0" />
+      <mass value="10.0" />
       <origin xyz="0 0 0" />
-      <inertia ixx="${0.0833333 * 1.0 * (0.3*0.3 + 0.2*0.2)}" ixy="0.0" ixz="0.0"
-        iyy="${0.0833333 * 1.0 * (0.4*0.4 + 0.2*0.2)}" iyz="0.0"
-        izz="${0.0833333 * 1.0 * (0.4*0.4 + 0.3*0.3)}" />
+      <inertia ixx="${0.0833333 * 10.0 * (0.3*0.3 + 0.2*0.2)}" ixy="0.0" ixz="0.0"
+        iyy="${0.0833333 * 10.0 * (0.4*0.4 + 0.2*0.2)}" iyz="0.0"
+        izz="${0.0833333 * 10.0 * (0.4*0.4 + 0.3*0.3)}" />
     </inertial>
 </link>
@@ -37,12 +37,4 @@
   <child link="base_link" />
   <origin xyz="0 0 0.1" />
-</joint>
-<!-- 2D LASER -->
-<link name="laser2d">
-</link>
-<joint name="laser2d_to_base_joint" type="fixed">
-  <parent link="base_link" />
-  <child link="laser2d" />
-  <origin xyz="0 0 0.2" />
 </joint>
 <!-- 3D LASER -->
@@ -78,5 +70,5 @@
           <max>100.0</max>
         </range>
-        <!-- <noise>
+        <noise>
           <type>uniform_dust</type>
           <hit_prob>0.0000001</hit_prob>
@@ -88,5 +80,5 @@
           <stddev>0.002</stddev>
           <range_exp>1.0</range_exp>
-        </noise> -->
+        </noise>
       </ray>
       <plugin name="rmagine_ros_laser3d" filename="librmagine_optix_ros_gzplugin.so">
