Commit message: added visuals for scanner. rmagine_ignore works for links now

File: urdf/robot_rotating_optix.urdf.xacro (robot description, xacro)
@@ -41,9 +41,15 @@
 <link name="laser2d">
   <collision>
-    <origin rpy="0 0 0" xyz="0 0 0.0"/>
+    <origin xyz="0.0 0.0 0.0" rpy="0 0 0"/>
     <geometry>
       <cylinder radius="0.0516" length="0.0717"/>
     </geometry>
   </collision>
+  <visual>
+    <origin xyz="0 0 0.0" rpy="0 0 0" />
+    <geometry>
+      <cylinder radius="0.0516" length="0.0717"/>
+    </geometry>
+  </visual>
   <inertial>
     <mass value="0.83"/>
@@ -54,4 +60,7 @@
   </inertial>
 </link>
+<gazebo reference="laser2d">
+  <rmagine_ignore/>
+</gazebo>
 <joint name="laser2d_to_base_joint" type="continuous">
   <parent link="base_link" />

File: urdf/robot_sensor_embree.urdf.xacro (robot description, xacro)
@@ -40,9 +40,31 @@
 <!-- 3D LASER -->
 <link name="laser3d">
+  <collision>
+    <origin rpy="0 0 0" xyz="0 0 0.0"/>
+    <geometry>
+      <cylinder radius="0.0516" length="0.0717"/>
+    </geometry>
+  </collision>
+  <visual>
+    <origin rpy="0 0 0" xyz="0 0 0.0"/>
+    <geometry>
+      <cylinder radius="0.0516" length="0.0717"/>
+    </geometry>
+  </visual>
+  <inertial>
+    <mass value="0.83"/>
+    <origin xyz="0.0 0.0 0.0"/>
+    <inertia ixx="${(0.83 * (3.0*0.0516*0.0516 + 0.0717*0.0717)) / 12.0}" ixy="0" ixz="0"
+      iyy="${(0.83 * (3.0*0.0516*0.0516 + 0.0717*0.0717)) / 12.0}" iyz="0"
+      izz="${0.5 * 0.83 * (0.0516*0.0516)}"/>
+  </inertial>
 </link>
+<gazebo reference="laser3d">
+  <rmagine_ignore/>
+</gazebo>
 <joint name="laser3d_to_base_joint" type="fixed">
   <parent link="base_link" />
   <child link="laser3d" />
-  <origin xyz="0 0 1.0" />
+  <origin xyz="0.0 0.0 0.5" />
 </joint>
 <gazebo reference="laser3d">
@@ -58,14 +80,14 @@
             <min_angle>${-M_PI}</min_angle>
             <increment>${1.0 * M_PI / 180.0}</increment>
-            <samples>360</samples>
+            <samples>1024</samples>
           </horizontal>
           <vertical>
-            <min_angle>${-60.0 * M_PI / 180.0}</min_angle>
+            <min_angle>${-45.0 * M_PI / 180.0}</min_angle>
             <increment>${2.0 * M_PI / 180.0}</increment>
-            <samples>60</samples>
+            <samples>45</samples>
           </vertical>
         </scan>
         <range>
-          <min>0.2</min>
+          <min>0.0</min>
           <max>100.0</max>
         </range>

File: urdf/robot_sensor_optix.urdf.xacro (robot description, xacro)
@@ -40,9 +40,31 @@
 <!-- 3D LASER -->
 <link name="laser3d">
+  <collision>
+    <origin rpy="0 0 0" xyz="0 0 0.0"/>
+    <geometry>
+      <cylinder radius="0.0516" length="0.0717"/>
+    </geometry>
+  </collision>
+  <visual>
+    <origin rpy="0 0 0" xyz="0 0 0.0"/>
+    <geometry>
+      <cylinder radius="0.0516" length="0.0717"/>
+    </geometry>
+  </visual>
+  <inertial>
+    <mass value="0.83"/>
+    <origin xyz="0.0 0.0 0.0"/>
+    <inertia ixx="${(0.83 * (3.0*0.0516*0.0516 + 0.0717*0.0717)) / 12.0}" ixy="0" ixz="0"
+      iyy="${(0.83 * (3.0*0.0516*0.0516 + 0.0717*0.0717)) / 12.0}" iyz="0"
+      izz="${0.5 * 0.83 * (0.0516*0.0516)}"/>
+  </inertial>
 </link>
+<gazebo reference="laser3d">
+  <rmagine_ignore/>
+</gazebo>
 <joint name="laser3d_to_base_joint" type="fixed">
   <parent link="base_link" />
   <child link="laser3d" />
-  <origin xyz="0 0 1.0" />
+  <origin xyz="0.0 0.0 0.5" />
 </joint>
 <gazebo reference="laser3d">
@@ -67,5 +89,5 @@
         </scan>
         <range>
-          <min>0.2</min>
+          <min>0.0</min>
           <max>100.0</max>
         </range>
@@ -97,40 +119,3 @@
     </sensor>
 </gazebo>
-<gazebo reference="laser3d">
-  <sensor type="gpu_ray" name="laser3d_gpu_old">
-    <always_on>true</always_on>
-    <update_rate>30</update_rate>
-    <pose>0 0 0 0 0 0</pose>
-    <visualize>false</visualize>
-    <ray>
-        <scan>
-            <horizontal>
-                <samples>1024</samples>
-                <resolution>1</resolution>
-                <min_angle>${-M_PI}</min_angle>
-                <max_angle>${M_PI}</max_angle>
-            </horizontal>
-            <vertical>
-                <samples>45</samples>
-                <resolution>1</resolution>
-                <min_angle>${-45.0 * M_PI / 180.0}</min_angle>
-                <max_angle>${43.0 * M_PI / 180.0}</max_angle>
-            </vertical>
-        </scan>
-        <range>
-            <min>0.2</min>
-            <max>100.0</max>
-            <resolution>0.01</resolution>
-        </range>
-    </ray>
-    <plugin name="laser3d_gpu_old_ros" filename="libgazebo_ros_velodyne_gpu_laser.so">
-      <topicName>old/pcl</topicName>
-      <frameName>laser3d</frameName>
-      <organize_cloud>false</organize_cloud>
-      <min_range>0.2</min_range>
-      <max_range>100.0</max_range>
-      <gaussianNoise>0.0</gaussianNoise>
-    </plugin>
-  </sensor>
-</gazebo>
 </robot>
