Commit message: added rotating scanner for embree and optix

File: urdf/robot_rotating_embree.urdf.xacro (robot description, xacro)
@@ -38,8 +38,8 @@
   <origin xyz="0 0 0.1" />
 </joint>
-<!-- 3D LASER -->
-<link name="laser3d">
+<!-- 2D  Rotating LASER -->
+<link name="laser2d">
   <collision>
-    <origin rpy="0 0 0" xyz="0 0 0.0"/>
+    <origin xyz="0.0 0.0 0.0" rpy="0 0 0"/>
     <geometry>
       <cylinder radius="0.0516" length="0.0717"/>
@@ -47,5 +47,5 @@
   </collision>
   <visual>
-    <origin rpy="0 0 0" xyz="0 0 0.0"/>
+    <origin xyz="0 0 0.0" rpy="0 0 0" />
     <geometry>
       <cylinder radius="0.0516" length="0.0717"/>
@@ -54,5 +54,5 @@
   <inertial>
     <mass value="0.83"/>
-    <origin xyz="0.0 0.0 0.0"/>
+    <origin xyz="0 0 0.0"/>
     <inertia ixx="${(0.83 * (3.0*0.0516*0.0516 + 0.0717*0.0717)) / 12.0}" ixy="0" ixz="0"
       iyy="${(0.83 * (3.0*0.0516*0.0516 + 0.0717*0.0717)) / 12.0}" iyz="0"
@@ -60,56 +60,41 @@
   </inertial>
 </link>
-<gazebo reference="laser3d">
+<gazebo reference="laser2d">
   <rmagine_ignore/>
 </gazebo>
-<joint name="laser3d_to_base_joint" type="fixed">
+<joint name="laser2d_to_base_joint" type="continuous">
   <parent link="base_link" />
-  <child link="laser3d" />
-  <origin xyz="0.0 0.0 0.5" />
+  <child link="laser2d" />
+  <origin xyz="0 0 0.5" rpy="${M_PI/2.0} 0.0 0.0" />
+  <axis xyz="0 1 0"/>
 </joint>
-<gazebo reference="laser3d">
-    <sensor type="rmagine_embree_spherical" name="laser3d">
+<gazebo reference="laser2d">
+    <sensor type="rmagine_embree_spherical" name="laser2d">
       <pose>0 0 0 0 0 0</pose>
       <always_on>true</always_on>
-      <update_rate>20</update_rate>
+      <update_rate>60</update_rate>
       <ray>
         <scan>
           <horizontal>
-            <min_angle>${-M_PI}</min_angle>
-            <increment>${1.0 * M_PI / 180.0}</increment>
-            <samples>1024</samples>
+            <min_angle>${-60.0 * M_PI / 180.0}</min_angle>
+            <increment>${0.01 * M_PI / 180.0}</increment>
+            <samples>12000</samples>
           </horizontal>
-          <vertical>
-            <min_angle>${-45.0 * M_PI / 180.0}</min_angle>
-            <increment>${2.0 * M_PI / 180.0}</increment>
-            <samples>45</samples>
-          </vertical>
         </scan>
         <range>
-          <min>0.0</min>
+          <min>0.2</min>
           <max>100.0</max>
         </range>
-        <noise>
-          <type>uniform_dust</type>
-          <hit_prob>0.0000001</hit_prob>
-          <return_prob>0.5</return_prob>
-        </noise>
-        <noise>
-          <type>rel_gaussian</type>
-          <mean>0.0</mean>
-          <stddev>0.002</stddev>
-          <range_exp>1.0</range_exp>
-        </noise>
       </ray>
       <plugin name="rmagine_ros_laser3d" filename="librmagine_embree_ros_gzplugin.so">
-          <frame>laser3d</frame>
+          <frame>laser2d</frame>
           <outputs>
+            <output name="scan">
+              <msg>sensor_msgs/LaserScan</msg>
+              <topic>laser2d/scan</topic>
+            </output>
             <output name="pcl">
               <msg>sensor_msgs/PointCloud</msg>
-              <topic>laser3d/pcl</topic>
-            </output>
-            <output name="pcl2">
-              <msg>sensor_msgs/PointCloud2</msg>
-              <topic>laser3d/pcl2</topic>
+              <topic>laser2d/pcl</topic>
             </output>
           </outputs>
@@ -117,3 +102,11 @@
     </sensor>
 </gazebo>
+<gazebo>
+  <plugin name="joint_state_publisher" filename="libgazebo_ros_joint_state_publisher.so">
+      <!-- <robotNamespace>/mm</robotNamespace> -->
+      <jointName>
+        robot_sensor::laser2d_to_base_joint
+      </jointName>
+  </plugin>
+</gazebo>
 </robot>

File: urdf/robot_rotating_optix.urdf.xacro (robot description, xacro)
@@ -74,6 +74,4 @@
       <always_on>true</always_on>
       <update_rate>60</update_rate>
-      <visualize>false</visualize>
-      <pre_alloc_mem>true</pre_alloc_mem>
       <ray>
         <scan>

File: urdf/robot_sensor_optix.urdf.xacro (robot description, xacro)
@@ -72,7 +72,5 @@
       <pose>0 0 0 0 0 0</pose>
       <always_on>true</always_on>
-      <update_rate>30</update_rate>
-      <visualize>false</visualize>
-      <pre_alloc_mem>true</pre_alloc_mem>
+      <update_rate>20</update_rate>
       <ray>
         <scan>
