Commit message: changed parameters so that they are a bit more similar to the default lidar_gpu plugin

File: urdf/example_robot.urdf.xacro (robot description, xacro)
@@ -98,4 +98,11 @@
     <origin xyz="0 0 ${wheel_radius - axis_height}" rpy="0 0 0"/>
   </joint>
+  <!-- base_footprint is deliberately massless (the standard ROS convention
+       for a ground-projected reference frame); sdformat's
+       preserveFixedJoint requires the preserved joint's parent link to
+       have its own <inertial>, so this one is left to lump normally (into
+       "base_footprint", which is already a real, expected TF frame via
+       DiffDrive's own odom->base_footprint output). Only lidar_joint below
+       needs preserving, so lidar_link survives as its own entity. -->
   <xacro:wheel name="wheel_front_left" x="${axis_front}" y="${wheel_y_offset}"/>
   <xacro:wheel name="wheel_front_right" x="${axis_front}" y="${-wheel_y_offset}"/>
@@ -121,4 +128,10 @@
     <origin xyz="0 0 ${body_height/2 + lidar_length/2 + 0.05}" rpy="0 0 0"/>
   </joint>
+  <!-- Keeps lidar_link a real, separate entity instead of being lumped
+       into base_link; see the comment above base_footprint_to_base_joint
+       for why the OTHER fixed joint here is deliberately left unpreserved. -->
+  <gazebo reference="lidar_joint">
+    <preserveFixedJoint>true</preserveFixedJoint>
+  </gazebo>
   <gazebo reference="lidar_link">
     <sensor name="lidar_sensor" type="custom" gz:type="rmagine_embree">
@@ -127,6 +140,10 @@
       <map_key>default</map_key>
       <frame>lidar_link</frame>
+      <!-- topic_points = topic_scan + "/points" matches gpu_lidar's own
+           auto-suffix convention (see README.md, "Migrating from
+           gpu_lidar"); keeps a bridge config written for a gpu_lidar
+           sensor working unchanged if this sensor ever swaps in for one. -->
       <topic_scan>/model/rmagine_example_robot/scan</topic_scan>
-      <topic_points>/model/rmagine_example_robot/points</topic_points>
+      <topic_points>/model/rmagine_example_robot/scan/points</topic_points>
       <range_min>0.15</range_min>
       <range_max>30.0</range_max>

Commit message: configurable URDF

File: urdf/example_robot.urdf.xacro (robot description, xacro)
@@ -10,9 +10,7 @@
   <xacro:include filename="$(find rmagine_gazebo_plugins)/urdf/wheel.urdf.xacro" />
   <!-- Args -->
-  <xacro:arg name="lidar3d" default="true"/>
-  <xacro:arg name="lidar2d" default="false"/>
-  <xacro:arg name="rgbd_camera" default="false"/>
+  <xacro:arg name="enable_gazebo_scan" default="true"/>
+  <xacro:arg name="rmagine_backend" default="embree"/>
   <xacro:property name="M_PI" value="3.14159265359"/>
-  <xacro:property name="imu_stdev" value="0.0001" />
   <xacro:property name="body_height" value="0.15"/>
   <xacro:property name="body_length" value="0.38"/>
@@ -109,36 +107,38 @@
   </joint>
   <gazebo reference="lidar3d">
-    <sensor name="lidar3d_gazebo_sensor" type="gpu_lidar">
-      <pose relative_to="lidar3d">0 0 0 0 0 0</pose>
-      <topic>/model/robot/lidar3d/gazebo</topic>
-      <update_rate>10</update_rate>
-      <ray>
-        <scan>
-          <horizontal>
-            <samples>360</samples>
-            <resolution>1</resolution>
-            <min_angle>${-M_PI}</min_angle>
-            <max_angle>${M_PI}</max_angle>
-          </horizontal>
-          <vertical>
-            <samples>16</samples>
+    <xacro:if value="$(arg enable_gazebo_scan)">
+      <sensor name="lidar3d_gazebo_sensor" type="gpu_lidar">
+        <pose relative_to="lidar3d">0 0 0 0 0 0</pose>
+        <topic>/model/robot/lidar3d/gazebo</topic>
+        <update_rate>10</update_rate>
+        <ray>
+          <scan>
+            <horizontal>
+              <samples>360</samples>
+              <resolution>1</resolution>
+              <min_angle>${-M_PI}</min_angle>
+              <max_angle>${M_PI}</max_angle>
+            </horizontal>
+            <vertical>
+              <samples>16</samples>
+              <resolution>0.01</resolution>
+              <min_angle>-${15.0 * M_PI/180.0}</min_angle>
+              <max_angle> ${15.0 * M_PI/180.0}</max_angle>
+            </vertical>
+          </scan>
+          <range>
+            <min>0.2</min>
+            <max>100.0</max>
             <resolution>0.01</resolution>
-            <min_angle>-${15.0 * M_PI/180.0}</min_angle>
-            <max_angle> ${15.0 * M_PI/180.0}</max_angle>
-          </vertical>
-        </scan>
-        <range>
-          <min>0.2</min>
-          <max>100.0</max>
-          <resolution>0.01</resolution>
-        </range>
-      </ray>
-      <always_on>1</always_on>
-      <visualize>true</visualize>
-      <frame_id>lidar3d</frame_id>
-      <gz_frame_id>lidar3d</gz_frame_id>
-      <ign_frame_id>lidar3d</ign_frame_id>
-    </sensor>
-    <sensor name="lidar3d_rmagine_sensor" type="custom" gz:type="rmagine_embree">
+          </range>
+        </ray>
+        <always_on>1</always_on>
+        <visualize>true</visualize>
+        <frame_id>lidar3d</frame_id>
+        <gz_frame_id>lidar3d</gz_frame_id>
+        <ign_frame_id>lidar3d</ign_frame_id>
+      </sensor>
+    </xacro:if>
+    <sensor name="lidar3d_rmagine_sensor" type="custom" gz:type="rmagine_$(arg rmagine_backend)">
       <always_on>true</always_on>
       <update_rate>20</update_rate>
